File: Arching_Civet/Arching_Civet.brd (EAGLE design)
At the start: 100 x 80 mm, 76 parts, among them IC1 OPA2134UA, IC2 OPA2134UA, Q1 J201, Q2 J201, Q3 J201, Q4 J201, Q5 J113

Commit message: Added brd sch
Added brd sch
Parts:
- moved R15 114.4 mm to (36.2, 12.3), flipped to the bottom, turned to 180 degrees
- moved C25 112.1 mm to (36.2, 10.9), flipped to the bottom, turned to 180 degrees
- moved C24 111.4 mm to (39.6, 11.8), flipped to the bottom, turned to 270 degrees
- moved R24 103.2 mm to (45.1, 14.4), turned to 180 degrees
- moved R25 101.3 mm to (39.0, 14.4)
- moved C22 99.9 mm to (32.1, 8.00)
- moved R10 98.7 mm to (42.4, 21.6), flipped to the bottom
- moved C23 97.6 mm to (32.0, 19.9), turned to 270 degrees
- moved R16 97.0 mm to (11.8, 11.8), turned to 90 degrees
- moved R27 92.4 mm to (20.6, 14.4)
- moved R12 92.2 mm to (29.6, 25.8), turned to 180 degrees
- moved R9 91.4 mm to (32.1, 12.4), turned to 90 degrees
- moved R13 89.8 mm to (10.9, 7.49), flipped to the bottom, turned to 90 degrees
- moved R14 89.5 mm to (5.08, 5.59), turned to 90 degrees
- moved R26 87.5 mm to (29.8, 33.0), turned to 180 degrees
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Routing:
- net VCC: track 0.00 -> 125.2 mm, vias 0 -> 2
- net GND: track 0.00 -> 52.6 mm, vias 0 -> 10
- net N$29: track 0.00 -> 41.4 mm
- net N$6: track 0.00 -> 41.2 mm, vias 0 -> 2
- net N$9: track 0.00 -> 38.9 mm, vias 0 -> 3
- net IN: track 0.00 -> 36.8 mm, vias 0 -> 1
- net PSIN: track 0.00 -> 33.6 mm, vias 0 -> 2
- net N$15: track 0.00 -> 31.6 mm, vias 0 -> 1
- net N$21: track 0.00 -> 30.0 mm, vias 0 -> 2
- net MVOL2: track 0.00 -> 28.9 mm
- net N$33: track 0.00 -> 28.6 mm
- net N$19: track 0.00 -> 27.1 mm
- net N$27: track 0.00 -> 27.0 mm
- net N$7: track 0.00 -> 26.5 mm
- net N$32: track 0.00 -> 25.2 mm, vias 0 -> 1
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- added copper zone on layer 1, net GND
- added copper zone on layer 16, net GND
Other:
- board size 100 x 80 mm -> 50.2 x 39.4 mm
- board text added: "+9V"
- board text added: "."
- board text added: "Arching Civet"
- board text added: "CAP_RETURN"
- board text added: "CAP_SEND"
- board text added: "GND"
- board text added: "IN"
- board text added: "MVOL2"
- board text added: "OUT"
- board text added: "PA_O"
- board text added: "PS_IN"
- board text added: "PS_O"
- board text added: "VDLINE"
